Commit message: added automatic center of mass calculations

File: examples/fancy_cube/flat.urdf (robot description, URDF)
Before this commit: robot flat, 1 links, 0 joints
Links:
- removed link flat
- added link _name, mass 1.0; collision mesh filename=flat/cube_flat_vhacd.obj scale=1 1 1; visual mesh filename=flat/cube_flat.obj scale=1 1 1

File: examples/fancy_cube/small_holder.urdf (robot description, URDF)
Before this commit: robot small_holder, 1 links, 0 joints
Links:
- removed link small_holder
- added link _name, mass 1.0; collision mesh filename=small_holder/holder_vhacd.obj scale=0.01 0.01 0.01; visual mesh filename=small_holder/holder.obj scale=0.01 0.01 0.01

File: examples/fancy_cube/textured.urdf (robot description, URDF)
Before this commit: robot textured, 1 links, 0 joints
Links:
- removed link textured
- added link _name, mass 1.0; collision mesh filename=textured/cube_tex_vhacd.obj scale=1 1 1; visual mesh filename=textured/cube_tex.obj scale=1 1 1

File: examples/ycb/006_mustard_bottle.urdf (robot description, URDF)
Before this commit: robot 006_mustard_bottle, 1 links, 0 joints
Links:
- removed link 006_mustard_bottle
- added link _name, mass 1.0; collision mesh filename=006_mustard_bottle/google_16k/textured_vhacd.obj scale=10 10 10; visual mesh filename=006_mustard_bottle/google_16k/textured.obj scale=10 10 10

File: examples/ycb/013_apple.urdf (robot description, URDF)
Before this commit: robot 013_apple, 1 links, 0 joints
Links:
- removed link 013_apple
- added link _name, mass 1.0; collision mesh filename=013_apple/google_16k/textured_vhacd.obj scale=10 10 10; visual mesh filename=013_apple/google_16k/textured.obj scale=10 10 10

File: examples/ycb/025_mug.urdf (robot description, URDF)
Before this commit: robot 025_mug, 1 links, 0 joints
Links:
- removed link 025_mug
- added link _name, mass 1.0; collision mesh filename=025_mug/google_16k/textured_vhacd.obj scale=10 10 10; visual mesh filename=025_mug/google_16k/textured.obj scale=10 10 10

File: examples/ycb/053_mini_soccer_ball.urdf (robot description, URDF)
Before this commit: robot 053_mini_soccer_ball, 1 links, 0 joints
Links:
- removed link 053_mini_soccer_ball
- added link _name, mass 1234.0; collision mesh filename=053_mini_soccer_ball/google_16k/textured_vhacd.obj scale=10 10 10; visual mesh filename=053_mini_soccer_ball/google_16k/textured.obj scale=10 10 10
